Commit message: Added robot3

File: urdf/robot1.urdf.xacro (robot description, xacro)
@@ -10,6 +10,6 @@
 		<child link="base_link" />
 	</joint>
+	<xacro:property name="base_l" value="1.5" />
 	<xacro:property name="base_w" value="1.5" />
-	<xacro:property name="base_l" value="1.5" />
 	<xacro:property name="base_h" value="0.1" />
 	<xacro:property name="base_m" value="5" />
@@ -18,5 +18,5 @@
 			<origin xyz="0 0 ${base_h/2}" rpy="0 0 0" />
 			<geometry>
-				<box size="${base_w} ${base_l} ${base_h}" />
+				<box size="${base_l} ${base_w} ${base_h}" />
 			</geometry>
 			<material name="blue"/>
@@ -25,5 +25,5 @@
 			<origin xyz="0 0 ${base_h/2}" rpy="0 0 0" />
 			<geometry>
-				<box size="${base_w} ${base_l} ${base_h}" />
+				<box size="${base_l} ${base_w} ${base_h}" />
 			</geometry>
 		</collision>
@@ -31,5 +31,5 @@
 			<origin xyz="0 0 ${base_h/2}" rpy="0 0 0" />
 			<mass value="${base_m}" />
-			<xacro:box_inertia m="${base_m}" x="${base_w}" y="${base_l}" z="${base_h}" />
+			<xacro:box_inertia m="${base_m}" x="${base_l}" y="${base_w}" z="${base_h}" />
 		</inertial>
 	</link>
@@ -38,9 +38,9 @@
 		<parent link="base_link" />
 		<child link="first_axis_link" />
-		<axis xyz="0 1 0" />
+		<axis xyz="1 0 0" />
 		<limit lower="${-base_l/2}" upper="${base_l/2}" velocity="100" effort="100" />
 	</joint>
+	<xacro:property name="first_l" value="0.2" />
 	<xacro:property name="first_w" value="0.2" />
-	<xacro:property name="first_l" value="0.2" />
 	<xacro:property name="first_h" value="0.2" />
 	<xacro:property name="first_m" value="0.5" />
@@ -49,5 +49,5 @@
 			<origin xyz="0 0 ${-first_h/2}" rpy="0 0 0" />
 			<geometry>
-				<box size="${first_w} ${first_l} ${first_h}" />
+				<box size="${first_l} ${first_w} ${first_h}" />
 			</geometry>
 			<material name="black"/>
@@ -56,5 +56,5 @@
 			<origin xyz="0 0 ${-first_h}" rpy="0 0 0" />
 			<geometry>
-				<box size="${first_w} ${first_l} ${first_h}" />
+				<box size="${first_l} ${first_w} ${first_h}" />
 			</geometry>
 		</collision>
@@ -62,5 +62,5 @@
 			<origin xyz="0 0 ${-first_h/2}" rpy="0 0 0" />
 			<mass value="${first_m}" />
-			<xacro:box_inertia m="${first_m}" x="${first_w}" y="${first_l}" z="${first_h}" />
+			<xacro:box_inertia m="${first_m}" x="${first_l}" y="${first_w}" z="${first_h}" />
 		</inertial>
 	</link>
@@ -69,5 +69,5 @@
 		<parent link="first_axis_link" />
 		<child link="second_axis_link" />
-		<axis xyz="0 1 0" />
+		<axis xyz="1 0 0" />
 		<limit lower="${-pi/2}" upper="${pi/2}" velocity="100" effort="100" />
 	</joint>
@@ -125,6 +125,6 @@
 		</inertial>
 	</link>
+	<xacro:property name="top_l" value="0.2" />
 	<xacro:property name="top_w" value="0.2" />
-	<xacro:property name="top_l" value="0.2" />
 	<xacro:property name="wheel_r" value="0.2" />
 	<xacro:property name="wheel_l" value="0.1" />
@@ -141,10 +141,10 @@
 				<origin xyz="0 0 ${-top_h/2}" rpy="0 0 0"/>
 				<geometry>
-					<box size="${top_w} ${top_l} ${top_h}" />
+					<box size="${top_l} ${top_w} ${top_h}" />
 				</geometry>
 				<material name="blue"/>
 			</visual>
 			<visual>
-				<origin xyz="0 0 ${-top_h-wheel_r}" rpy="0 ${pi/2} 0"/>
+				<origin xyz="0 0 ${-top_h-wheel_r}" rpy="${pi/2} 0 0"/>
 				<geometry>
 					<cylinder radius="${wheel_r}" length="${wheel_l}" />
@@ -155,5 +155,5 @@
 				<origin xyz="0 0 ${-top_h/2-wheel_r}" rpy="0 0 0"/>
 				<geometry>
-					<box size="${top_w} ${2*wheel_r} ${top_h+2*wheel_r}" />
+					<box size="${top_l} ${2*wheel_r} ${top_h+2*wheel_r}" />
 				</geometry>
 			</collision>
@@ -165,7 +165,7 @@
 		</link>
 	</xacro:macro>
-	<xacro:wheel prefix="fl" x="${-base_w/2+top_w/2}" y="${base_l/2-top_l/2}" />
-	<xacro:wheel prefix="bl" x="${-base_w/2+top_w/2}" y="${-base_l/2+top_l/2}" />
-	<xacro:wheel prefix="fr" x="${base_w/2-top_w/2}" y="${base_l/2-top_l/2}" />
-	<xacro:wheel prefix="br" x="${base_w/2-top_w/2}" y="${-base_l/2+top_l/2}" />
+	<xacro:wheel prefix="fl" x="${base_l/2-top_w/2}" y="${base_w/2-top_l/2}" />
+	<xacro:wheel prefix="bl" x="${-base_l/2+top_w/2}" y="${base_w/2-top_l/2}" />
+	<xacro:wheel prefix="fr" x="${base_l/2-top_w/2}" y="${-base_w/2+top_l/2}" />
+	<xacro:wheel prefix="br" x="${-base_l/2+top_w/2}" y="${-base_w/2+top_l/2}" />
 </robot>

File: urdf/robot3.urdf.xacro (robot description, xacro)
@@ -41,7 +41,7 @@
 		<limit lower="${-base_l/2}" upper="${base_l/2}" velocity="100" effort="100" />
 	</joint>
+	<xacro:property name="first_l" value="0.2" />
 	<xacro:property name="first_w" value="0.2" />
-	<xacro:property name="first_l" value="0.2" />
-	<xacro:property name="first_h" value="0.2" />
+	<xacro:property name="first_h" value="0.8" />
 	<xacro:property name="first_m" value="0.5" />
 	<link name="first_axis_link">
@@ -49,5 +49,5 @@
 			<origin xyz="0 0 ${-first_h/2}" rpy="0 0 0" />
 			<geometry>
-				<box size="${first_w} ${first_l} ${first_h}" />
+				<box size="${first_l} ${first_w} ${first_h}" />
 			</geometry>
 			<material name="black"/>
@@ -56,5 +56,5 @@
 			<origin xyz="0 0 ${-first_h}" rpy="0 0 0" />
 			<geometry>
-				<box size="${first_w} ${first_l} ${first_h}" />
+				<box size="${first_l} ${first_w} ${first_h}" />
 			</geometry>
 		</collision>
@@ -62,9 +62,9 @@
 			<origin xyz="0 0 ${-first_h/2}" rpy="0 0 0" />
 			<mass value="${first_m}" />
-			<xacro:box_inertia m="${first_m}" x="${first_w}" y="${first_l}" z="${first_h}" />
+			<xacro:box_inertia m="${first_m}" x="${first_l}" y="${first_w}" z="${first_h}" />
 		</inertial>
 	</link>
 	<joint name="second_axis_joint" type="revolute">
-		<origin xyz="0 0 ${-first_h}" rpy="0 0 0" />
+		<origin xyz="0 0 ${-first_h}" rpy="${pi/2} 0 0" />
 		<parent link="first_axis_link" />
 		<child link="second_axis_link" />
@@ -72,10 +72,10 @@
 		<limit lower="${-pi/2}" upper="${pi/2}" velocity="100" effort="100" />
 	</joint>
-	<xacro:property name="arm_length" value="0.6" />
-	<xacro:property name="arm_radius" value="0.05" />
-	<xacro:property name="arm_mass" value="1" />
+	<xacro:property name="arm_length" value="0.4" />
+	<xacro:property name="arm_radius" value="0.07" />
+	<xacro:property name="arm_mass" value="5.3" />
 	<link name="second_axis_link">
 		<visual>
-			<origin xyz="0 0 ${-arm_length/2}" rpy="0 0 0" />
+			<origin xyz="0 0 0" rpy="0 0 0" />
 			<geometry>
 				<cylinder length="${arm_length}" radius="${arm_radius}" />
@@ -84,5 +84,5 @@
 		</visual>
 		<collision>
-			<origin xyz="0 0 ${-arm_length/2}" rpy="0 0 0" />
+			<origin xyz="0 0 0" rpy="0 0 0" />
 			<geometry>
 				<cylinder length="${arm_length}" radius="${arm_radius}" />
@@ -90,21 +90,23 @@
 		</collision>
 		<inertial>
-			<origin xyz="0 0 ${-arm_length/2}" rpy="0 0 0" />
+			<origin xyz="0 0 0" rpy="0 0 0" />
 			<mass value="${arm_mass}" />
 			<xacro:cylinder_inertia m="${arm_mass}" r="${arm_radius}" h="${arm_length}" />
 		</inertial>
 	</link>
-	<xacro:property name="arm2_radius" value="0.05" />
-	<xacro:property name="arm2_length" value="0.6" />
-	<xacro:property name="arm2_mass" value="0.5" />
-	<joint name="third_axis_joint" type="continuous">
-		<origin xyz="0 0 ${-arm_length}" rpy="0 0 0" />
+	<xacro:property name="arm2_radius" value="0.03" />
+	<xacro:property name="arm2_length" value="0.8" />
+	<xacro:property name="arm2_mass" value="1.4" />
+	<xacro:property name="arm2_stroke" value="0.3" />
+	<joint name="third_axis_joint" type="prismatic">
+		<origin xyz="0 0 0" rpy="0 0 0" />
 		<parent link="second_axis_link" />
 		<child link="third_axis_link" />
-		<axis xyz="1 0 0" />
+		<axis xyz="0 0 1" />
+		<limit lower="${-arm2_stroke}" upper="${arm2_stroke}" velocity="100" effort="100" />
 	</joint>
 	<link name="third_axis_link">
 		<visual>
-			<origin xyz="0 0 ${-arm2_length/2}" rpy="0 0 0" />
+			<origin xyz="0 0 0" rpy="0 0 0" />
 			<geometry>
 				<cylinder length="${arm2_length}" radius="${arm2_radius}" />
@@ -113,5 +115,5 @@
 		</visual>
 		<collision>
-			<origin xyz="0 0 ${-arm2_length/2}" rpy="0 0 0" />
+			<origin xyz="0 0 0" rpy="0 0 0" />
 			<geometry>
 				<cylinder length="${arm2_length}" radius="${arm2_radius}" />
@@ -119,5 +121,5 @@
 		</collision>
 		<inertial>
-			<origin xyz="0 0 ${-arm2_length/2}" rpy="0 0 0" />
+			<origin xyz="0 0 0" rpy="0 0 0" />
 			<mass value="${arm2_mass}" />
 			<xacro:cylinder_inertia m="${arm2_mass}" r="${arm2_radius}" h="${arm2_length}" />
